File: powerdistribution/powerdistribution.kicad_sch (KiCad schematic)
At the start: 11 parts, among them J1 Conn_01x02_Socket, J2 Conn_01x02_Socket, J3 Conn_01x02_Socket, J4 Screw_Terminal_01x02, J5 Screw_Terminal_01x02, J6 Conn_01x10_Socket, J7 Conn_01x10_Socket, SW1 RA1H1C112R, SW2 RA1H1C112R, U1 BQ7790512PW

Commit message: BMS draft
Parts:
- added C1, C2, C3, C4, C5, C6: C, symbol Device:C
- added R1, R2, R3, R4, R5: R_US, symbol Device:R_US
Connections:
- net Vdd: now reaches U1.1 (VDD)
- net Vdd: now also C6.2, R5.2
- net AVdd: now reaches U1.17 (CCFG)
- net AVdd: now also U1.2 (AVDD), C5.1
- net GND: now reaches U1.18 (CTRC)
- net GND: now also BT1.1-, U1.19 (CTRD), U1.20 (DVSS), U1.3 (VC5), U1.4 (VC4), U1.8 (AVSS), C1.2, C2.2, C3.2, C4.1, C4.2, C5.2, C6.1, R4.2
- net at U1.5 (VC3): now also C3.1, R3.2
- net at U1.6 (VC2): now also C2.1, R2.2
- net at U1.7 (VC1): now also C1.1, R1.2
- net at BT1.1+: now also BT1.2-, R1.1
- net at BT1.2+: now also BT1.3-, R2.1
- net at BT1.3+: now also BT1.4-, R3.1
- net Pack+: now reaches BT1.4+
- net Pack+: now also R4.1, R5.1
Other:
- moved on the sheet: BT1, U1

Commit message: pwr draft
Parts:
- added IC1: STEF01FTR, SOP65P640X120-15N, symbol HPRsymbols:STEF01FTR
- added MOSFET1: T2N7002AK_LM, SOT23_TOS, symbol HPRsymbols:T2N7002AK_LM
- added R6, R7, R8: R_US, symbol Device:R_US
- added RT1: 103AT-2, 103AT2, symbol HPRsymbols:103AT-2
Connections:
- net GND: now also U1.9 (SRP), R7.1, RT1.2; no longer C4.1, R4.2, U1.3 (VC5), U1.4 (VC4)
- net at U1.10 (SRN): now also R7.2
- net at U1.14 (LD): now also R6.2
- net at U1.15 (TS): now also R8.1, RT1.1
- net at U1.16 (VTB): now also R8.2
- new net: C4.1, R4.2, U1.3 (VC5), U1.4 (VC4)
- new net Pack-: R6.1
Other:
- moved on the sheet: C1, C2, C3, C5, C6, J4, J5, U1

Commit message: efuse draft
Parts:
- removed MOSFET1: T2N7002AK_LM, SOT23_TOS, symbol HPRsymbols:T2N7002AK_LM
- added C7, C8, C9: C, symbol Device:C
- added Q1, Q2: IRLML0030, Package_TO_SOT_SMD:SOT-23, symbol Transistor_FET:IRLML0030
- added R10, R11, R12, R13, R14, R9: R, symbol Device:R
Connections:
- net GND: now also IC1.3 (GND), IC1.4 (AUTO), C7.1, C8.2, C9.2, R10.2, R12.2
- net at IC1.1 (UVLO): now also R11.1, R12.1
- net at IC1.10 (I-LIMIT): now also R14.1
- net Efuse_fault: now reaches IC1.12 (EN/FAULT)
- net at IC1.13 (PG): now also R13.1
- net Vin_efuse: now reaches IC1.14 (VCC)
- net Vin_efuse: now also IC1.15 (EPAD), C8.1, R11.2, R13.2
- net at IC1.2 (DV/DT): now also C7.2
- net at IC1.5 (VCLAMP): now also R10.1, R9.2
- net Vout_efuse: now reaches IC1.6 (VOUT_1)
- net Vout_efuse: now also IC1.7 (VOUT_2), IC1.8 (VOUT_3), IC1.9 (VOUT_4), C9.1, R14.2, R9.1
Other:
- moved on the sheet: IC1

Commit message: efuse and bms pcb draft
Parts:
- removed C1, C2, C3, C4: C, symbol Device:C
- removed R1, R2, R3, R4: R_US, symbol Device:R_US
- added C1, C2, C3, C4: JMK105BJ105KV-F, HPRfootprints:CAPC1005X55N, symbol HPRsymbols:JMK105BJ105KV-F
- added R1, R2, R3, R4: 1K, HPRfootprints:R0402, symbol HPRsymbols:SMD-RES-1K-5_-1_16W_0402_
- added R15, R16, R17, R18: R_US, symbol Device:R_US
- BT1: footprint BK-18650-PC8:BAT_BK-18650-PC8 -> HPRfootprints:BAT_BK-18650-PC8
- IC1: footprint SOP65P640X120-15N -> HPRfootprints:SOP65P640X120-15N
- RT1: footprint 103AT2 -> HPRfootprints:103AT2
- U1: footprint BQ7790512PW:SOP65P640X120-20N -> HPRfootprints:SOP65P640X120-20N
Connections:
- net GND: now also C1.2, C2.2, C3.2, C4.1
- net Pack+: now also R4.1
- net Pack-: now also Q2.2 (S), R16.2
- net at Q2.1 (G): now also R16.1, R18.2
- net at Q2.3 (D): now also Q1.3 (D)
- net at U1.3 (VC5), U1.4 (VC4): now also C4.2, R4.2
- net at BT1.3+, BT1.4-: now also R3.1
- net at U1.5 (VC3): now also C3.1, R3.2
- net sns-: now reaches R7.2, U1.10 (SRN)
- net sns-: now also Q1.2 (S), R15.2
- net at U1.11 (DSG): now also R17.1
- net at U1.13 (CHG): now also R18.1
- net at U1.6 (VC2): now also C2.1, R2.2
- net at U1.7 (VC1): now also C1.1, R1.2
- net at Q1.1 (G): now also R15.1, R17.2
- net at BT1.2+, BT1.3-: now also R2.1
- net at BT1.1+, BT1.2-: now also R1.1
Other:
- moved on the sheet: Q1, Q2

Commit message: draft
Parts:
- removed R5: R_US, symbol Device:R_US
- added R5: 1K, HPRfootprints:R0402, symbol HPRsymbols:SMD-RES-1K-5_-1_16W_0402_
Connections:
- net Pack+: now also R5.2
- net Vdd: now also R5.1
Changed lines of the file:
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@@
+	)
+	(junction
+		(at 54.61 68.58)
+		(diameter 0)
+		(color 0 0 0 0)
 	)
 	(junction
@@
 	(junction
 		(at 205.74 100.33)
-		(diameter 0)
-		(color 0 0 0 0)
-	)
-	(junction
-		(at 54.61 68.58)
 		(diameter 0)
 		(color 0 0 0 0)
@@
 	)
 	(symbol
-		(lib_id "Device:R_US")
-		(at 54.61 72.39 0)
-		(unit 1)
-		(exclude_from_sim no)
-		(in_bom yes)
-		(on_board yes)
-		(dnp no)
-		(fields_autoplaced yes)
-		(property "Reference" "R5"
-			(at 57.15 71.1199 0)
-			(effects
-				(font
-					(size 1.27 1.27)
-				)
-				(justify left)
-			)
-		)
-		(property "Value" "R_US"
-			(at 57.15 73.6599 0)
-			(effects
-				(font
-					(size 1.27 1.27)
-				)
-				(justify left)
-			)
-		)
-		(property "Footprint" ""
-			(at 55.626 72.644 90)
-			(effects
-				(font
-					(size 1.27 1.27)
-				)
-				(hide yes)
-			)
-		)
-		(property "Datasheet" "~"
-			(at 54.61 72.39 0)
-			(effects
-				(font
-					(size 1.27 1.27)
-				)
-				(hide yes)
-			)
-		)
-		(property "Description" "Resistor, US symbol"
-			(at 54.61 72.39 0)
-			(effects
-				(font
-					(size 1.27 1.27)
-				)
-				(hide yes)
-			)
-		)
-		(pin "1"
-		)
-		(pin "2"
-		)
-		(instances
-			(project ""
-				(path "/4cf67788-0fe7-4c87-8363-3433eaa0df90"
-					(reference "R5")
-					(unit 1)
-				)
-			)
-		)
-	)
-	(symbol
 		(lib_id "Transistor_FET:IRLML0030")
 		(at 185.42 55.88 270)
@@
 					(unit 1)
 				)
+			)
+		)
+	)
+	(symbol
+		(lib_id "HPRsymbols:SMD-RES-1K-5_-1_16W_0402_")
+		(at 54.61 72.39 90)
+		(unit 1)
+		(exclude_from_sim no)
+		(in_bom yes)
+		(on_board yes)
+		(dnp no)
+		(fields_autoplaced yes)
+		(property "Reference" "R5"
+			(at 55.88 72.3899 90)
+			(effects
+				(font
+					(size 1.27 1.27)
+				)
+				(justify right)
+			)
+		)
+		(property "Value" "1K"
+			(at 54.61 72.39 0)
+			(effects
+				(font
+					(size 1.27 1.27)
+				)
+				(justify bottom)
+				(hide yes)
+			)
+		)
+		(property "Footprint" "HPRfootprints:R0402"
+			(at 54.61 72.39 0)
+			(effects
+				(font
+					(size 1.27 1.27)
+				)
+				(justify bottom)
+				(hide yes)
+			)
+		)
+		(property "Datasheet" ""
+			(at 54.61 72.39 0)
+			(effects
+				(font
+					(size 1.27 1.27)
+				)
+				(hide yes)
+			)
+		)
+		(property "Description" ""
+			(at 54.61 72.39 0)
+			(effects
+				(font
+					(size 1.27 1.27)
+				)
+				(hide yes)
+			)
+		)
+		(property "MPN" "RC0402JR-071KL"
+			(at 54.61 72.39 0)
+			(effects
+				(font
+					(size 1.27 1.27)
+				)
+				(justify bottom)
+				(hide yes)
+			)
+		)
+		(pin "1"
+		)
+		(pin "2"
+		)
+		(instances
+			(project "powerdistribution"
+				(path "/4cf67788-0fe7-4c87-8363-3433eaa0df90"
+					(reference "R5")
+					(unit 1)
+				)

Commit message: added buck converters into schematic
Parts:
- removed J1, J2, J3: Conn_01x02_Socket, symbol Connector:Conn_01x02_Socket
- removed J6, J7: Conn_01x10_Socket, symbol Connector:Conn_01x10_Socket
- added 100nf, 100nf1, 100nf2: C, symbol Device:C
- added C10, C11, C16, C17, C23, C24: 22 uf, symbol Device:C_Small
- added C10, C15, C22: 22uf, symbol Device:C_Small
- added C11, C18, C25: 2.7nf, symbol Device:C
- added C12, C19, C26: 10 nf, symbol Device:C_Small
- added C13, C14, C20, C21, C27, C28: 10 uf, symbol Device:C_Small
- added L1, L3: 6.8 uh, symbol Device:L
- added L2: 4.7uh, symbol Device:L
- added R19, R22, R25: 10k, symbol Device:R_US
- added R20, R26: 52.3, symbol Device:R_US
- added R21, R27: 15.8k, symbol Device:R_US
- added R23: 31.6k, symbol Device:R_US
- added R24: 10.5k, symbol Device:R_US
- added U2, U3, U4: AP64501QSP-13, SO-8EP_DIO, symbol 2025-11-16_06-05-29:AP64501QSP-13
Connections:
- net Pack- is gone; now on net GND: Q2.2 (S), R16.2, R6.1
- net GND: now also C12.1, C13.2, C14.2, C19.1, C20.2, C21.2, C26.1, C27.2, C28.2, R19.1, R25.1
- net Pack+: now also C13.1, C14.1, C20.1, C21.1, C27.1, C28.1, U2.2 (VIN), U2.3 (EN), U3.2 (VIN), U3.3 (EN), U4.2 (VIN), U4.3 (EN)
- new net: 100nf.2, L1.1, U4.8 (SW)
- new net: C11.1, R24.2
- new net: R22.2, R23.1, U2.5 (FB)
- new net: R27.1, U4.6 (COMP)
- new net: C25.1, R27.2
- new net: 100nf1.2, L2.1, U2.8 (SW)
- new net: 100nf2.2, L3.1, U3.8 (SW)
- new net: C19.2, U3.4 (SS)
- new net: R25.2, R26.1, U4.5 (FB)
- new net: C26.2, U4.4 (SS)
- new net: 100nf2.1, U3.1 (BST)
- new net: R19.2, R20.1, U3.5 (FB)
- new net: R21.1, U3.6 (COMP)
- new net: C18.1, R21.2
- new net: C12.2, U2.4 (SS)
- new net: 100nf.1, U4.1 (BST)
- new net: R24.1, U2.6 (COMP)
- new net: 100nf1.1, U2.1 (BST)
- new net 3.3v_output: C10.2, C10.2, C11.2, L2.2, R23.2
- new net 5v_output: C22.2, C23.2, C24.2, L1.2, R26.2
- new net 6v_output: C15.2, C16.2, C17.2, L3.2, R20.2
- new net GNDREF: C10.1, C10.1, C11.1, C11.2, C15.1, C16.1, C17.1, C18.2, C22.1, C23.1, C24.1, C25.2, U2.7 (GND), U3.7 (GND), U4.7 (GND)
Other:
- moved on the sheet: BT1, C1, C2, C3, C4, C5, C6, C7, C8, C9, IC1, J4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

Commit message: organization, still schematic errors
Parts:
- added C29, C30, C31, C32, C33, C34: C, symbol Device:C
- added IC2, IC3: STEF01FTR, HPRfootprints:SOP65P640X120-15N, symbol HPRsymbols:STEF01FTR
- added J1, J2: 282837-2, HPRfootprints:TE_282837-2, symbol HPRsymbols:282837-2
- added J3: M20-6102045, RHDR40W66P254_2X20_5146X500X1105P, symbol HPRlibrary:M20-6102045
- added Q3 (x2): MMBT3904, Package_TO_SOT_SMD:SOT-23, symbol Transistor_BJT:MMBT3904
- added Q4: SI4925DDY-T1-GE3, HPRfootprints:SOIC127P600X175-8N, symbol HPRsymbols:SI4925DDY-T1-GE3
- added R28, R29, R30, R31, R32, R33, R34, R35, R36, R37, R38, R39: R, symbol Device:R
- added R40, R41: 1K, Resistor_SMD:R_0603_1608Metric_Pad0.98x0.95mm_HandSolder, symbol Device:R
- added R42, R43: 10K, Resistor_SMD:R_0603_1608Metric_Pad0.98x0.95mm_HandSolder, symbol Device:R
- added TP4, TP5, TP6, TP7: TestPoint, TestPoint:TestPoint_Pad_1.0x1.0mm, symbol Connector:TestPoint
- 100nf1, C10, C11, C12, C13, C14, L2, R22, R23, R24, U2: now not fitted
Connections:
- net Efuse_fault: now also IC2.12 (EN/FAULT), IC3.12 (EN/FAULT)
- net GND: now also R22.1, C29.1, C30.2, C31.2, C32.1, C33.2, C34.2, IC2.3 (GND), IC2.4 (AUTO), IC3.3 (GND), IC3.4 (AUTO), J1.2, J2.2, Q3.2 (E), Q3.2 (E), R28.2, R30.2, R34.2, R36.2
- net Vin_efuse: now also C31.1, C34.1, IC2.14 (VCC), IC2.15 (EPAD), IC3.14 (VCC), IC3.15 (EPAD), R31.2, R32.2, R37.2, R38.2
- net Vout_efuse: now also C30.1, C33.1, IC2.6 (VOUT_1), IC2.7 (VOUT_2), IC2.8 (VOUT_3), IC2.9 (VOUT_4), IC3.6 (VOUT_1), IC3.7 (VOUT_2), IC3.8 (VOUT_3), IC3.9 (VOUT_4), R29.1, R33.2, R35.1, R39.2
- new net: Q3.1 (B), R41.2, TP4.1
- new net: Q3.3 (C), Q4.2 (G1), R42.2
- new net: IC2.5 (VCLAMP), R28.1, R29.2
- new net: IC3.1 (UVLO), R36.1, R37.1
- new net: IC2.1 (UVLO), R30.1, R31.1
- new net: IC2.10 (I-LIMIT), R33.1
- new net: IC2.13 (PG), R32.1
- new net: C29.2, IC2.2 (DV/DT)
- new net: IC3.5 (VCLAMP), R34.1, R35.2
- new net: IC3.10 (I-LIMIT), R39.1
- new net: IC3.13 (PG), R38.1
- new net: C32.2, IC3.2 (DV/DT)
- new net: Q3.3 (C), Q4.4 (G2), R43.2
- new net: Q3.1 (B), R40.2, TP5.1
- new net: J1.1, Q4.7 (D1_1), Q4.8 (D1_2), TP6.1
- new net: J2.1, Q4.5 (D2_1), Q4.6 (D2_2), TP7.1
- new net PYRO1: R40.1
- new net PYRO2: R41.1
- new net VBATT: Q4.1 (S1), Q4.3 (S2), R42.1, R43.1
Other:
- note added: "3.3V Buck [DNP]"
- note added: "5V Buck"
- note added: "6V Buck"
- note added: "BMS"
- note added: "E-Fuse"
- note added: "E-Fuse [DNP]"
- note added: "PYRO"
- moved on the sheet: 100nf, 100nf2, BT1, C1, C15, C16, C17, C18, C19, C2, C20, C21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
