File: powerdistribution/powerdistribution.kicad_sch (KiCad schematic)
At the start: 99 parts, among them J1 282837-2, J2 282837-2, J3 M20-6102045, Q1 IRLML0030, Q2 IRLML0030, Q3 IRLML0030, Q5 IRLML0030, U1 BQ7790512PW, U2 AP64501QSP-13, U3 AP64501QSP-13, U4 AP64501QSP-13, U5 TPS1HC30BQPWPRQ1, U6 TPS1HC30BQPWPRQ1, U7 ESP32-DEVKIT-V1

Commit message: reorganization, need to update pyros, reconsider charging, assign nets to pins, think how pin switch will be mounted
Parts:
- added C36: 100nF, Capacitor_SMD:C_0603_1608Metric_Pad1.08x0.95mm_HandSolder, symbol Device:C
- added C39, C40: 10uF, Capacitor_SMD:C_0603_1608Metric_Pad1.08x0.95mm_HandSolder, symbol Device:C
- added C41: 22uF, Capacitor_SMD:C_0603_1608Metric_Pad1.08x0.95mm_HandSolder, symbol Device:C
- added R37, R38: 10k, Resistor_SMD:R_0603_1608Metric_Pad0.98x0.95mm_HandSolder, symbol Device:R_US
- added R39: 1.2k, Resistor_SMD:R_0603_1608Metric_Pad0.98x0.95mm_HandSolder, symbol Device:R
- added R45: 4.7k, Resistor_SMD:R_0603_1608Metric_Pad0.98x0.95mm_HandSolder, symbol Device:R
- added TP3, TP4: TestPoint, Connector_PinHeader_2.00mm:PinHeader_1x01_P2.00mm_Vertical, symbol Connector:TestPoint
- added TP5, TP6: TestPoint, Connector_PinHeader_2.54mm:PinHeader_1x01_P2.54mm_Vertical, symbol Connector:TestPoint
- added U8: LD1117S50TR_SOT223, Package_TO_SOT_SMD:SOT-223-3_TabPin2, symbol Regulator_Linear:LD1117S50TR_SOT223
- added U9: MIC29302AWD-TR, HPRfootprints:TO-252-5_MCH, symbol HPRsymbols:MIC29302AWD-TR
- R13: value 65k -> 31.6k
- R19: value 65k -> 52.3k
Connections:
- net 6V: now also C41.1, R45.2, TP6.1, U9.4 (OUT); no longer C29.1, C30.1, C31.1, L3.1, R19.1
- net GND: now also C36.2, C39.2, C40.2, C41.2, R39.2, U8.1 (GND), U9.3 (GND), U9.6 (GND)
- net Pack+: now also C36.1, U8.3 (VI)
- net 5V_EN: now reaches R28.1, TP2.1
- net 5V_EN: now also R29.1, TP4.1
- net at C26.2, C27.2, U2.2 (VIN)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: no longer U5.10 (VOUT__1), U5.9 (VOUT)
- net 6V_DIAGEN: now reaches R26.1
- net 6V_DIAGEN: now also TP3.1
- net 6V_EN: now reaches R21.1, TP1.1
- net 5V: now reaches U7.30 (VIN)
- net 5V: now also C29.1, C30.1, C31.1, L3.1, R19.1
- new net: C40.1, U5.10 (VOUT__1), U5.9 (VOUT), U9.1 (EN), U9.2 (IN)
- new net: R39.1, R45.1, U9.5 (ADJ)
- new net: R37.1, R38.2
- new net LDO_5V: C39.1, TP5.1, U8.2 (VO)
Other:
- note added: "5A Switch"
- note added: "5V LDO"
- note added: "6V 3A LDO Linear Regulator"
- note added: "Excluded schematics"
- note added: "Headers and Ports"
- note added: "PIN SWITCH TO ENABLE"
- note removed: "3.3V LDO"
- note removed: "PIN SWITCH"
- note removed: "Switch"
- moved on the sheet: C10, C15, C16, C26, C27, C6, C7, C8, C9, L1, R10, R11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

Commit message: power should be ok now? need to look at BMS, pyro, connectors, remaining nets..
Parts:
- added C42, C43: 1uF, Capacitor_SMD:C_0603_1608Metric_Pad1.08x0.95mm_HandSolder, symbol Device:C
- added IC1: NCP718ASNADJT1G, HPRlibrary:NCP718_SOT95P280X100-5N, symbol HPRlibrary:NCP718ASNADJT1G
- added R46, R47, R48, R49, R50, R51: 10k, Resistor_SMD:R_0603_1608Metric_Pad0.98x0.95mm_HandSolder, symbol Device:R_US
- added R52, R53: 0, Resistor_SMD:R_0603_1608Metric_Pad0.98x0.95mm_HandSolder, symbol Device:R_US
- added R54: 19k, Resistor_SMD:R_0603_1608Metric_Pad0.98x0.95mm_HandSolder, symbol Device:R_US
- added R55: 6k, Resistor_SMD:R_0603_1608Metric_Pad0.98x0.95mm_HandSolder, symbol Device:R_US
- R37: now not fitted
Connections:
- net 5V: now also R52.1; no longer U7.30 (VIN)
- net 5V_EN: now also R48.1, R49.2
- net 6V_DIAGEN: now also R46.1, R47.2
- net 6V_EN: now also R37.1, R38.2
- net GND: now also R38.1, C42.2, C43.2, IC1.2 (GND), R47.1, R49.1, R51.1, R55.1
- net LDO_5V: now also R37.2, C43.1, IC1.5 (OUT), R46.2, R48.2, R50.2, R53.1, R54.2
- net Pack+: now also C42.1, IC1.1 (IN), IC1.3 (EN)
- net at U7.16 (EN): now also U7.30 (VIN), R52.2, R53.2
- new net: IC1.4 (NC/ADJ), R54.1, R55.2
- new net 5V_DIAGEN: R50.1, R51.2
- no-connect marks 0 -> 6
Other:
- moved on the sheet: C36, C39, R38, TP5, U8

Commit message: placement draft 1
Parts:
- IC1: footprint HPRlibrary:NCP718_SOT95P280X100-5N -> HPRfootprints:NCP718_SOT95P280X100-5N
- L2, L3: footprint (none) -> Inductor_SMD:L_0603_1608Metric_Pad1.05x0.95mm_HandSolder
- U3, U4: footprint HPRlibrary:SO-8EP_DIO-L -> HPRfootprints:SO-8EP_DIO-L
- U5, U6: footprint HPRlibrary:IC_TPS1HC30BQPWPRQ1 -> HPRfootprints:IC_TPS1HC30BQPWPRQ1
- U7: footprint HPRlibrary:MODULE_ESP32_DEVKIT_V1 -> HPRfootprints:MODULE_ESP32_DEVKIT_V1
Connections:
- net 5V_DIAGEN: now also R29.1, TP4.1
- net 5V_EN: no longer R29.1, TP4.1
Changed lines of the file:
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@@
 	)
 	(junction
-		(at 490.22 101.6)
-		(diameter 0)
-		(color 0 0 0 0)
-	)
-	(junction
 		(at 351.79 314.96)
 		(diameter 0)
@@
 	)
 	(junction
+		(at 490.22 101.6)
+		(diameter 0)
+		(color 0 0 0 0)
+	)
+	(junction
 		(at 162.56 175.26)
 		(diameter 0)
@@
 		)
 	)
-	(label "5V_EN"
+	(label "5V_DIAGEN"
 		(at 69.85 328.93 0)
 		(effects
@@
 	)
 	(symbol
-		(lib_id "Device:C")
-		(at 435.61 102.87 0)
-		(unit 1)
-		(exclude_from_sim no)
-		(in_bom yes)
-		(on_board no)
-		(dnp no)
-		(fields_autoplaced yes)
-		(property "Reference" "C42"
-			(at 439.42 101.5999 0)
-			(effects
-				(font
-					(size 1.27 1.27)
-				)
-				(justify left)
-			)
-		)
-		(property "Value" "1uF"
-			(at 439.42 104.1399 0)
-			(effects
-				(font
-					(size 1.27 1.27)
-				)
-				(justify left)
-			)
-		)
-		(property "Footprint" "Capacitor_SMD:C_0603_1608Metric_Pad1.08x0.95mm_HandSolder"
-			(at 436.5752 106.68 0)
-			(effects
-				(font
-					(size 1.27 1.27)
-				)
-				(hide yes)
-			)
-		)
-		(property "Datasheet" "~"
-			(at 435.61 102.87 0)
-			(effects
-				(font
-					(size 1.27 1.27)
-				)
-				(hide yes)
-			)
-		)
-		(property "Description" "Unpolarized capacitor"
-			(at 435.61 102.87 0)
-			(effects
-				(font
-					(size 1.27 1.27)
-				)
-				(hide yes)
-			)
-		)
-		(pin "2"
-		)
-		(pin "1"
-		)
-		(instances
-			(project "powerdistribution"
-				(path "/4cf67788-0fe7-4c87-8363-3433eaa0df90"
-					(reference "C42")
-					(unit 1)
-				)
-			)
-		)
-	)
-	(symbol
 		(lib_id "Device:C_Small")
 		(at 234.95 337.82 0)
@@
 			)
 		)
-		(property "Footprint" "HPRlibrary:IC_TPS1HC30BQPWPRQ1"
+		(property "Footprint" "HPRfootprints:IC_TPS1HC30BQPWPRQ1"
 			(at 114.3 170.18 0)
 			(effects
@@
 			)
 		)
-		(property "Footprint" "HPRlibrary:SO-8EP_DIO-L"
+		(property "Footprint" "HPRfootprints:SO-8EP_DIO-L"
 			(at 247.65 323.85 0)
 			(effects
@@
 	)
 	(symbol
+		(lib_id "Device:C")
+		(at 490.22 105.41 0)
+		(unit 1)
+		(exclude_from_sim no)
+		(in_bom yes)
+		(on_board yes)
+		(dnp no)
+		(fields_autoplaced yes)
+		(property "Reference" "C43"
+			(at 494.03 104.1399 0)
+			(effects
+				(font
+					(size 1.27 1.27)
+				)
+				(justify left)
+			)
+		)
+		(property "Value" "1uF"
+			(at 494.03 106.6799 0)
+			(effects
+				(font
+					(size 1.27 1.27)
+				)
+				(justify left)
+			)
+		)
+		(property "Footprint" "Capacitor_SMD:C_0603_1608Metric_Pad1.08x0.95mm_HandSolder"
+			(at 491.1852 109.22 0)
+			(effects
+				(font
+					(size 1.27 1.27)
+				)
+				(hide yes)
+			)
+		)
+		(property "Datasheet" "~"
+			(at 490.22 105.41 0)
+			(effects
+				(font
+					(size 1.27 1.27)
+				)
+				(hide yes)
+			)
+		)
+		(property "Description" "Unpolarized capacitor"
+			(at 490.22 105.41 0)
+			(effects
+				(font
+					(size 1.27 1.27)
+				)
+				(hide yes)
+			)
+		)
+		(pin "1"
+		)
+		(pin "2"
+		)
+		(instances
+			(project ""
+				(path "/4cf67788-0fe7-4c87-8363-3433eaa0df90"
+					(reference "C43")
+					(unit 1)
+				)
+			)
+		)
+	)
+	(symbol
 		(lib_id "Device:C_Small")
 		(at 232.41 256.54 0)
@@
 			)
 		)
-		(property "Footprint" "HPRlibrary:NCP718_SOT95P280X100-5N"
+		(property "Footprint" "HPRfootprints:NCP718_SOT95P280X100-5N"
 			(at 476.25 193.98 0)
 			(effects
@@
 	)
 	(symbol
+		(lib_id "Device:C")
+		(at 435.61 102.87 0)
+		(unit 1)
+		(exclude_from_sim no)
+		(in_bom yes)
+		(on_board yes)
+		(dnp no)
+		(fields_autoplaced yes)
+		(property "Reference" "C42"
+			(at 439.42 101.5999 0)
+			(effects
+				(font
+					(size 1.27 1.27)
+				)
+				(justify left)
+			)
+		)
+		(property "Value" "1uF"
+			(at 439.42 104.1399 0)
+			(effects
+				(font
+					(size 1.27 1.27)
+				)
+				(justify left)
+			)
+		)
+		(property "Footprint" "Capacitor_SMD:C_0603_1608Metric_Pad1.08x0.95mm_HandSolder"
+			(at 436.5752 106.68 0)
+			(effects
+				(font
+					(size 1.27 1.27)
+				)
+				(hide yes)
+			)
+		)
+		(property "Datasheet" "~"
+			(at 435.61 102.87 0)
+			(effects
+				(font
+					(size 1.27 1.27)
+				)
+				(hide yes)
+			)
+		)
+		(property "Description" "Unpolarized capacitor"
+			(at 435.61 102.87 0)
+			(effects
+				(font
+					(size 1.27 1.27)
+				)
+				(hide yes)
+			)
+		)
+		(pin "1"
+		)
+		(pin "2"
+		)
+		(instances
+			(project ""
+				(path "/4cf67788-0fe7-4c87-8363-3433eaa0df90"
+					(reference "C42")
+					(unit 1)
+				)
+			)
+		)
+	)
+	(symbol
 		(lib_id "Device:R")
 		(at 309.88 52.07 90)
@@
 			)
 		)
-		(property "Footprint" "HPRlibrary:MODULE_ESP32_DEVKIT_V1"
+		(property "Footprint" "HPRfootprints:MODULE_ESP32_DEVKIT_V1"
 			(at 487.68 182.88 0)
 			(effects
@@
 			)
 		)
-		(property "Footprint" "HPRlibrary:IC_TPS1HC30BQPWPRQ1"
+		(property "Footprint" "HPRfootprints:IC_TPS1HC30BQPWPRQ1"
 			(at 114.3 328.93 0)
 			(effects
@@
 	)
 	(symbol
-		(lib_id "Device:C")
-		(at 490.22 105.41 0)
-		(unit 1)
-		(exclude_from_sim no)
-		(in_bom yes)
-		(on_board no)
-		(dnp no)
-		(fields_autoplaced yes)
-		(property "Reference" "C43"
-			(at 494.03 104.1399 0)
-			(effects
-				(font
-					(size 1.27 1.27)
-				)
-				(justify left)
-			)
-		)
-		(property "Value" "1uF"
-			(at 494.03 106.6799 0)
-			(effects
-				(font
-					(size 1.27 1.27)
-				)
-				(justify left)
-			)
-		)
-		(property "Footprint" "Capacitor_SMD:C_0603_1608Metric_Pad1.08x0.95mm_HandSolder"
-			(at 491.1852 109.22 0)
-			(effects
-				(font
-					(size 1.27 1.27)
-				)
-				(hide yes)
-			)
-		)
-		(property "Datasheet" "~"
-			(at 490.22 105.41 0)
-			(effects
-				(font
-					(size 1.27 1.27)
-				)
-				(hide yes)
-			)
-		)
-		(property "Description" "Unpolarized capacitor"
-			(at 490.22 105.41 0)
-			(effects
-				(font
-					(size 1.27 1.27)
-				)
-				(hide yes)
-			)
-		)
-		(pin "2"
-		)
-		(pin "1"
-		)
-		(instances
-			(project "powerdistribution"
-				(path "/4cf67788-0fe7-4c87-8363-3433eaa0df90"
-					(reference "C43")
-					(unit 1)
-				)
-			)
-		)
-	)
-	(symbol
 		(lib_id "power:GND")
 		(at 90.17 67.31 0)
@@
 			)
 		)
-		(property "Footprint" ""
+		(property "Footprint" "Inductor_SMD:L_0603_1608Metric_Pad1.05x0.95mm_HandSolder"
 			(at 316.23 307.34 0)
 			(effects
@@
 			)
 		)
-		(property "Footprint" "HPRlibrary:SO-8EP_DIO-L"
+		(property "Footprint" "HPRfootprints:SO-8EP_DIO-L"
 			(at 245.11 242.57 0)
 			(effects
@@
 			)
 		)
-		(property "Footprint" ""
+		(property "Footprint" "Inductor_SMD:L_0603_1608Metric_Pad1.05x0.95mm_HandSolder"
 			(at 313.69 226.06 0)
 			(effects
